Commit message: collision information and joint limits added

File: urdf/aironbot.urdf (robot description, URDF)
Before this commit: robot aironbot, 2 links, 1 joints
Links:
- link base_link: mass None -> 1; geometry collision mesh filename=package://aironbot_description/meshes/manipulator_base_link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; visual mesh filename=package://aironbot_description/meshes/manipulator_base_link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
- link link_1: mass None -> 1; geometry collision mesh filename=package://aironbot_description/meshes/manipulator_link.stl; visual mesh filename=package://aironbot_description/meshes/manipulator_link.stl
Joints:
- joint link_1_to_base: limit (none) -> lower=-1.57 upper=1.57 effort=1000.0 velocity=0.5; type continuous -> revolute

Commit message: inertia removed

File: urdf/aironbot.urdf (robot description, URDF)
Before this commit: robot aironbot, 2 links, 1 joints
Links:
- link base_link: mass 1 -> None
- link link_1: mass 1 -> None
